Commit message: model update and system launch

File: gazebo_c_pkg/models/crazyflie_xacro/crazyflie.urdf.xacro (robot description, xacro)
@@ -1,131 +1,113 @@
 <?xml version="1.0"?>
 <robot name="crazyflie" xmlns:xacro="http://www.ros.org/wiki/xacro">
-  <link name="crazyflie/body">
-    <pose> 0 0 17.425E-3 0 0 0</pose>
+  <link name="world">
+    <origin xyz="0 0 0" rpy="0 0 0"/>
+  </link>
+  <!-- Main body -->
+  <link name="crazyflie_body">
     <inertial>
-      <mass>0.025</mass>
-      <inertia>
-        <ixx>16.571710E-06</ixx>
-        <iyy>16.655602E-06</iyy>
-        <izz>29.261652E-06</izz>
-        <ixy>0.830806E-06</ixy>
-        <ixz>0.718277E-06</ixz>
-        <iyz>1.800197E-06</iyz>
-      </inertia>
+      <mass value="0.027"/>
+      <origin xyz="0 0 0" rpy="0 0 0"/>
+      <inertia ixx="0.000016571710" ixy="0.000000830806" ixz="0.000000718277"
+               iyy="0.000016655602" iyz="0.000001800197" izz="0.000029261652"/>
     </inertial>
-    <collision name="crazyflie/body_collision">
+    <collision>
+      <origin xyz="0 0 0.017425" rpy="0 0 0"/>
       <geometry>
-        <box>
-          <size>0.10 0.10 34.850E-3</size>
-        </box>
+        <box size="0.10 0.10 0.03485"/>
       </geometry>
     </collision>
-    <visual name="crazyflie/body_visual">
+    <visual>
+      <origin xyz="0 0 0.017425" rpy="0 0 0"/>
       <geometry>
-        <mesh>
-          <uri>package://gazebo_c_pkg/models/crazyflie_xacro/meshes/collada_files/cf2_assembly.dae</uri>
-        </mesh>
+        <mesh filename="package://gazebo_c_pkg/models/crazyflie_xacro/meshes/collada_files/cf2_assembly.dae"/>
       </geometry>
     </visual>
   </link>
-  <link name="crazyflie/m1_prop">
-    <pose>0.031 -0.031 0.021 0 0 0</pose>
+  <!-- Propeller 1 -->
+  <link name="crazyflie_m1_prop">
     <inertial>
-      <mass>0.0008</mass>
-      <inertia>
-        <ixx>8.33333E-09</ixx>
-        <iyy>1.08333E-07</iyy>
-        <izz>1.13333E-07</izz>
-      </inertia>
+      <mass value="0.0008"/>
+      <origin xyz="0 0 0" rpy="0 0 0"/>
+      <inertia ixx="8.33333e-09" ixy="0" ixz="0"
+               iyy="1.08333e-07" iyz="0" izz="1.13333e-07"/>
     </inertial>
-    <visual name="crazyflie/m1_visual">
+    <visual>
+      <origin xyz="0.031 -0.031 0.021" rpy="0 0 0"/>
       <geometry>
-        <mesh>
-          <uri>package://gazebo_c_pkg/models/crazyflie_xacro/meshes/collada_files/ccw_prop.dae</uri>
-        </mesh>
+        <mesh filename="package://gazebo_c_pkg/models/crazyflie_xacro/meshes/collada_files/ccw_prop.dae"/>
       </geometry>
     </visual>
   </link>
-  <link name="crazyflie/m2_prop">
-    <pose>-0.031 -0.031 0.021 0 0 0</pose>
+  <!-- Propeller 2 -->
+  <link name="crazyflie_m2_prop">
     <inertial>
-      <mass>0.0008</mass>
-      <inertia>
-        <ixx>8.33333E-09</ixx>
-        <iyy>1.08333E-07</iyy>
-        <izz>1.13333E-07</izz>
-      </inertia>
+      <mass value="0.0008"/>
+      <origin xyz="0 0 0" rpy="0 0 0"/>
+      <inertia ixx="8.33333e-09" ixy="0" ixz="0"
+               iyy="1.08333e-07" iyz="0" izz="1.13333e-07"/>
     </inertial>
-    <visual name="crazyflie/m2_visual">
+    <visual>
+      <origin xyz="-0.031 -0.031 0.021" rpy="0 0 0"/>
       <geometry>
-        <mesh>
-          <uri>package://gazebo_c_pkg/models/crazyflie_xacro/meshes/collada_files/cw_prop.dae</uri>
-        </mesh>
+        <mesh filename="package://gazebo_c_pkg/models/crazyflie_xacro/meshes/collada_files/cw_prop.dae"/>
       </geometry>
     </visual>
   </link>
-  <link name="crazyflie/m3_prop">
-    <pose>-0.031 0.031 0.021 0 0 0</pose>
+  <!-- Propeller 3 -->
+  <link name="crazyflie_m3_prop">
     <inertial>
-      <mass>0.0008</mass>
-      <inertia>
-        <ixx>8.33333E-09</ixx>
-        <iyy>1.08333E-07</iyy>
-        <izz>1.13333E-07</izz>
-      </inertia>
+      <mass value="0.0008"/>
+      <origin xyz="0 0 0" rpy="0 0 0"/>
+      <inertia ixx="8.33333e-09" ixy="0" ixz="0"
+               iyy="1.08333e-07" iyz="0" izz="1.13333e-07"/>
     </inertial>
-    <visual name="crazyflie/m3_visual">
+    <visual>
+      <origin xyz="-0.031 0.031 0.021" rpy="0 0 0"/>
       <geometry>
-        <mesh>
-          <uri>package://gazebo_c_pkg/models/crazyflie_xacro/meshes/collada_files/ccw_prop.dae</uri>
-        </mesh>
+        <mesh filename="package://gazebo_c_pkg/models/crazyflie_xacro/meshes/collada_files/ccw_prop.dae"/>
       </geometry>
     </visual>
   </link>
-  <link name="crazyflie/m4_prop">
-    <pose>0.031 0.031 0.021 0 0 0</pose>
+  <!-- Propeller 4 -->
+  <link name="crazyflie_m4_prop">
     <inertial>
-      <mass>0.0008</mass>
-      <inertia>
-        <ixx>8.33333E-09</ixx>
-        <iyy>1.08333E-07</iyy>
-        <izz>1.13333E-07</izz>
-      </inertia>
+      <mass value="0.0008"/>
+      <origin xyz="0 0 0" rpy="0 0 0"/>
+      <inertia ixx="8.33333e-09" ixy="0" ixz="0"
+               iyy="1.08333e-07" iyz="0" izz="1.13333e-07"/>
     </inertial>
-    <visual name="crazyflie/m4_visual">
+    <visual>
+      <origin xyz="0.031 0.031 0.021" rpy="0 0 0"/>
       <geometry>
-        <mesh>
-          <uri>package://gazebo_c_pkg/models/crazyflie_xacro/meshes/collada_files/cw_prop.dae</uri>
-        </mesh>
+        <mesh filename="package://gazebo_c_pkg/models/crazyflie_xacro/meshes/collada_files/cw_prop.dae"/>
       </geometry>
     </visual>
   </link>
-  <joint name="crazyflie/m1_joint" type="fixed">
-    <child>crazyflie/m1_prop</child>
-    <parent>crazyflie/body</parent>
-    <axis>
-      <xyz>0 0 1</xyz>
-    </axis>
+  <!-- Joints -->
+  <joint name="base_joint" type="fixed">
+    <parent link="world"/>
+    <child link="crazyflie_body"/>
+    <origin xyz="0 0 1" rpy="0 0 0"/>
   </joint>
-  <joint name="crazyflie/m2_joint" type="fixed">
-    <child>crazyflie/m2_prop</child>
-    <parent>crazyflie/body</parent>
-    <axis>
-      <xyz>0 0 1</xyz>
-    </axis>
+  <joint name="m1_joint" type="fixed">
+    <parent link="crazyflie_body"/>
+    <child link="crazyflie_m1_prop"/>
+    <origin xyz="0.0 0.0 0.0" rpy="0 0 0"/>
   </joint>
-  <joint name="crazyflie/m3_joint" type="fixed">
-    <child>crazyflie/m3_prop</child>
-    <parent>crazyflie/body</parent>
-    <axis>
-      <xyz>0 0 1</xyz>
-    </axis>
+  <joint name="m2_joint" type="fixed">
+    <parent link="crazyflie_body"/>
+    <child link="crazyflie_m2_prop"/>
+    <origin xyz="-0.031 -0.031 0.021" rpy="0 0 0"/>
   </joint>
-  <joint name="crazyflie/m4_joint" type="fixed">
-    <child>crazyflie/m4_prop</child>
-    <parent>crazyflie/body</parent>
-    <axis>
-      <xyz>0 0 1</xyz>
-    </axis>
+  <joint name="m3_joint" type="fixed">
+    <parent link="crazyflie_body"/>
+    <child link="crazyflie_m3_prop"/>
+    <origin xyz="-0.031 0.031 0.021" rpy="0 0 0"/>
+  </joint>
+  <joint name="m4_joint" type="fixed">
+    <parent link="crazyflie_body"/>
+    <child link="crazyflie_m4_prop"/>
+    <origin xyz="0.031 0.031 0.021" rpy="0 0 0"/>
   </joint>
 </robot>
